Commit message: Updates

File: test/integration/fixed_joint_reduction_visual.urdf (robot description, URDF)
Before this commit: robot fixed_joint_reduction_test_odel, 8 links, 7 joints
Links:
- removed link link1a
- removed link link2
- removed link link2a
- removed link link3
- removed link link3a
Joints:
- removed joint joint01a
- removed joint joint12
- removed joint joint12a
- removed joint joint23
- removed joint joint23a
