Commit message: Add collisions to fixed_joint_reduction.urdf

File: test/integration/fixed_joint_reduction.urdf (robot description, URDF)
Before this commit: robot fixed_joint_reduction_test_odel, 8 links, 7 joints
Links:
- link link0: geometry collision box size=0.1 0.1 1.0; visual box size=0.1 0.1 1.0
- link link1: geometry collision box size=0.2 3.0 0.2; visual box size=0.2 3.0 0.2
- link link1a: geometry collision box size=0.2 3.0 0.2; visual box size=0.2 3.0 0.2
- link link2: geometry collision box size=0.3 0.3 2.0; visual box size=0.3 0.3 2.0
- link link2a: geometry collision box size=0.3 0.3 2.0; visual box size=0.3 0.3 2.0
- link link3: geometry collision box size=0.3 0.4 0.5; visual box size=0.3 0.4 0.5
- link link3a: geometry collision box size=0.3 0.4 0.5; visual box size=0.3 0.4 0.5
