Commit message: test and fix reduction for collisions and visuals.

File: test/integration/fixed_joint_reduction_collision_extension.urdf (robot description, URDF)
Before this commit: robot lumping_test, 2 links, 1 joints
Links:
- added link child_link_1a, mass 1.0; collision sphere radius=0.03; visual sphere radius=0.03
- added link child_link_2, mass 1.0; collision sphere radius=0.05; visual sphere radius=0.05
- link base_link: geometry collision sphere radius=0.02; visual sphere radius=0.02
Joints:
- added joint fixed_joint_1a: type fixed, parent base_link, child child_link_1a, origin xyz=0 0 0 rpy=0 0 0
- added joint fixed_joint_2: type fixed, parent child_link_1, child child_link_2, origin xyz=0 0 0 rpy=0 0 0
