Commit message: Fix up the provide_feedback test to be correct.
As mentioned in issue #77, this test is actually not doing
much at the moment, mostly because the links don't have
inertia.  However, nobody ever noticed this fact because
the test itself was too weak.  Take the proposed patch
from issue #77, apply it, and then fix up the URDF so
that we actually test the correct thing.

File: test/integration/provide_feedback.urdf (robot description, URDF)
Before this commit: robot provide_feedback_test, 4 links, 3 joints
Links:
- link link0: mass None -> 0.5
- link link1: mass None -> 0.5
- link link2: mass None -> 0.5
