Commit message: Fix cfm damping integration test for URDF.
Must like for provide_feedback, make sure we are actually
parsing things properly inside the test, and then fix the
URDF to have inertial for the link so we hit those tests.

File: test/integration/cfm_damping_implicit_spring_damper.urdf (robot description, URDF)
Before this commit: robot cfm_damping_implicit_spring_damper_conversion_test, 5 links, 4 joints
Links:
- link link0: mass None -> 0.5
- link link1: mass None -> 0.5
- link link2: mass None -> 0.5
- link link3: mass None -> 0.5
